File: flightcontroller.kicad_pcb (KiCad board)
At the start: 2 copper layers, 24.6 x 27.4 mm, 3 parts, among them SW1 1571983-4, U1 MS561101BA03-50, U2 XMC1302T028X0016ABXUMA1

Commit message: Add files via upload
Parts:
- added U3: TLV70233DSER, TLV70233DSER:DSE0006A, F.Cu at (135.8, 111.7)
- moved U1 0.72 mm to (140.8, 107.8)
Connections:
- U1 pad 8: Net-(U1-SCLK) -> unconnected-(U1-SCLK-Pad8)
- U2 pad 1: Net-(U1-SCLK) -> unconnected-(U2-IN1/AN-Pad1)
Routing:
- net Net-(U1-SCLK): track 4.76 -> 0.00 mm
